File: PCB/StanzaBoard/StanzaBoard.kicad_sch (KiCad schematic)
At the start: 2 parts, among them U1 STM32L432KCU6, U2 ESP32-S3-WROOM-1-N8

Commit message: Progressing PCB devboard version
Parts:
- added C1, C17, C31, C4, C5, C50, C53: 10uF, Capacitor_SMD:C_0805_2012Metric, symbol Device:C
- added C10: 10uF, Capacitor_SMD:CP_Elec_5x5.4, symbol Device:C_Polarized
- added C11: 100pF, Capacitor_SMD:C_0603_1608Metric, symbol Device:C
- added C12, C15, C16: 1nF, Capacitor_SMD:C_0603_1608Metric, symbol Device:C
- added C13: 47uF, Capacitor_SMD:CP_Elec_5x5.4, symbol Device:C_Polarized
- added C14, C58, C59: 2.2nF, Capacitor_SMD:C_0603_1608Metric, symbol Device:C
- added C18, C20, C21, C25, C32, C41, C43, C51, C52, C54, C6: 100nF, Capacitor_SMD:C_0603_1608Metric, symbol Device:C
- added C2, C24, C3, C33, C57: 1uF, Capacitor_SMD:C_0603_1608Metric, symbol Device:C
- added C22, C40, C42: 4.7uF, Capacitor_SMD:C_0805_2012Metric, symbol Device:C
- added C23: 10nF, Capacitor_SMD:C_0603_1608Metric, symbol Device:C
- added C30: 22uF, Capacitor_SMD:C_0805_2012Metric, symbol Device:C
- added C55, C56: 2.2uF, Capacitor_SMD:C_0603_1608Metric, symbol Device:C
- added D1: PWR (green), LED_SMD:LED_0603_1608Metric, symbol Device:LED
- added D2: BAT54S, Package_TO_SOT_SMD:SOT-23, symbol Diode:BAT54S
- added D3: STATUS, LED_SMD:LED_0603_1608Metric, symbol Device:LED
- added F1: 500mA hold, Fuse:Fuse_1206_3216Metric, symbol Device:Polyfuse
- added FB1, FB2, FB3: 600R, Inductor_SMD:L_0603_1608Metric, symbol Device:FerriteBead
- added J1: USB4105-GF-A, Connector_USB:USB_C_Receptacle_GCT_USB4105-xx-A_16P_TopMnt_Horizontal, symbol Connector:USB_C_Receptacle_USB2.0_16P
- added J2: Guitar In 6.35mm, Connector_Audio:Jack_6.35mm_Neutrik_NMJ4HCD2_Horizontal, symbol Connector_Audio:AudioJack2
- added J3: Line Out 6.35mm TRS, Connector_Audio:Jack_6.35mm_Neutrik_NMJ6HCD2_Horizontal, symbol Connector_Audio:AudioJack3
- added J4: SWD (VDD,SWCLK,GND,SWDIO,NRST,SWO), Connector_PinHeader_2.54mm:PinHeader_1x06_P2.54mm_Vertical, symbol Connector_Generic:Conn_01x06
- added NT1: NetTie AGND-GND, NetTie:NetTie-2_SMD_Pad0.5mm, symbol Device:NetTie_2
- added Q1, Q2: MMBT3904, Package_TO_SOT_SMD:SOT-23, symbol Transistor_BJT:MMBT3904
- added R1, R2: 5.1k, Resistor_SMD:R_0603_1608Metric, symbol Device:R
- added R10, R11: 2.2M, Resistor_SMD:R_0603_1608Metric, symbol Device:R
- added R12, R18, R19, R20, R30, R31, R32, R33, R50: 10k, Resistor_SMD:R_0603_1608Metric, symbol Device:R
- added R13: 3k, Resistor_SMD:R_0603_1608Metric, symbol Device:R
- added R14: 220R, Resistor_SMD:R_0603_1608Metric, symbol Device:R
- added R15, R16: 6.8k, Resistor_SMD:R_0603_1608Metric, symbol Device:R
- added R17, R24, R3, R42: 1k, Resistor_SMD:R_0603_1608Metric, symbol Device:R
- added R21, R22, R23, R34, R35, R36: 33R, Resistor_SMD:R_0603_1608Metric, symbol Device:R
- added R40: 22.1k, Resistor_SMD:R_0603_1608Metric, symbol Device:R
- added R41: 47.5k, Resistor_SMD:R_0603_1608Metric, symbol Device:R
- added R51, R52: 470R, Resistor_SMD:R_0603_1608Metric, symbol Device:R
- added SW1: RESET, Button_Switch_SMD:SW_SPST_TL3342, symbol Switch:SW_Push
- added SW2: BOOT, Button_Switch_SMD:SW_SPST_TL3342, symbol Switch:SW_Push
- added TP1: SAI_MCLK, TestPoint:TestPoint_Pad_D1.0mm, symbol Connector:TestPoint
- added unit 2 of U1
- added U3: TL974, Package_SO:SOIC-14_3.9x8.7mm_P1.27mm, symbol Amplifier_Operational:TL074
- added U4: USBLC6-2SC6, Package_TO_SOT_SMD:SOT-23-6, symbol Power_Protection:USBLC6-2SC6
- added U5: AP2112K-3.3, Package_TO_SOT_SMD:SOT-23-5, symbol Regulator_Linear:AP2112K-3.3
- added U6: CP2102N-A02-GQFN28, Package_DFN_QFN:QFN-28-1EP_5x5mm_P0.5mm_EP3.35x3.35mm, symbol Interface_USB:CP2102N-Axx-xQFN28
- added U7: PCM5102A, Package_SO:TSSOP-20_4.4x6.5mm_P0.65mm, symbol Audio:PCM5102A
Connections:
- net GND: now reaches U2.1 (GND)
- net GND: now also U2.40 (GND), U2.41 (GND), U2.42 (GND), U2.43 (GND), U2.44 (GND), U2.45 (GND), U2.46 (GND), U2.47 (GND), U2.48 (GND), U2.49 (GND), C1.2, C2.2, C20.2, C21.2, C22.2, C23.2, C24.2, C25.2, C3.2, C30.2, C31.2, C32.2, C33.2, C4.2, C40.2, C41.2, C42.2, C43.2, C50.2, C51.2, C52.2, C53.2, C54.2, C56.2, C57.2, C58.2, C59.2, D1.1 (K), D3.1 (K), J1.A1 (GND), J1.A12 (GND), J1.B1 (GND), J1.B12 (GND), J1.S1 (SHIELD), J3.S, J4.3 (Pin_3), NT1.1, R1.2, R2.2, R20.2, R41.2, SW1.2, SW2.2, U1.16 (VSS), U1.32 (VSS), U4.2 (GND), U5.2 (GND), U6.29 (GND), U6.3 (GND), U7.10 (DEMP), U7.11 (FLT), U7.12 (SCK), U7.16 (FMT), U7.19 (DGND), U7.3 (CPGND), U7.9 (AGND)
- net I2S_SD: now reaches U2.10 (IO17)
- net I2S_SD: now also R23.2
- net ESP_DAC_BCK: now reaches U2.18 (IO10)
- net ESP_DAC_BCK: now also R34.1
- net ESP_DAC_LRCK: now reaches U2.19 (IO11)
- net ESP_DAC_LRCK: now also R35.1
- net +3V3: now reaches U2.2 (3V3)
- net +3V3: now also C20.1, C21.1, C22.1, C3.1, C30.1, C31.1, C32.1, C4.1, C53.1, C54.1, FB2.1, FB3.1, J4.1 (Pin_1), R3.1, R30.1, R31.1, R50.1, U1.1 (VDD), U1.17 (VDD), U5.5 (VOUT), U7.20 (DVDD)
- net ESP_DAC_DIN: now reaches U2.20 (IO12)
- net ESP_DAC_DIN: now also R36.1
- net ESP_IO0: now reaches U2.27 (IO0)
- net ESP_IO0: now also Q2.3 (C), R31.2, SW2.1
- net ESP_EN: now reaches U2.3 (EN)
- net ESP_EN: now also C33.1, Q1.3 (C), R30.2, SW1.1
- net ESP_RXD: now reaches U2.36 (RXD0)
- net ESP_RXD: now also U6.26 (TXD)
- net ESP_TXD: now reaches U2.37 (TXD0)
- net ESP_TXD: now also U6.25 (RXD)
- net I2S_BCLK: now reaches U2.8 (IO15)
- net I2S_BCLK: now also R21.2
- net I2S_WS: now reaches U2.9 (IO16)
- net I2S_WS: now also R22.2
- net STM_SAI_SCK: now reaches U1.18 (PA8)
- net STM_SAI_SCK: now also R21.1
- net STM_SAI_FS: now reaches U1.19 (PA9)
- net STM_SAI_FS: now also R22.1
- net STM_SAI_SD: now reaches U1.20 (PA10)
- net STM_SAI_SD: now also R23.1
- net SWDIO: now reaches U1.23 (PA13)
- net SWDIO: now also J4.4 (Pin_4)
- net SWCLK: now reaches U1.24 (PA14)
- net SWCLK: now also J4.2 (Pin_2)
- net SWO_LED: now reaches U1.26 (PB3)
- net SWO_LED: now also J4.6 (Pin_6), R24.1
- net BOOT0: now reaches U1.31 (PH3-BOOT0)
- net BOOT0: now also R20.1
- net NRST: now reaches U1.4 (NRST)
- net NRST: now also C25.1, J4.5 (Pin_5)
- net ADC_IN: now reaches U1.6 (PA0-CK_IN)
- net ADC_IN: now also C16.1, D2.3 (COM), R17.2
- net STM_MCLK: now reaches U1.9 (PA3)
- net STM_MCLK: now also TP1.1
- new net +3.3VA: C23.1, C24.1, D2.2 (K), FB2.2, R18.1, U1.5 (VDDA/VREF+)
- new net +3V3_DAC: C50.1, C51.1, C52.1, FB3.2, U7.1 (CPVDD), U7.8 (AVDD)
- new net +5V: C1.1, C2.1, C40.1, C41.1, F1.2, FB1.1, U5.1 (VIN), U5.3 (EN), U6.7 (VREGIN)
- new net +5VA: C18.1, C5.1, C6.1, FB1.2, U3.4 (V+)
- new net AA_OUT: C14.2, R17.1, U3.8, U3.9 (-)
- new net AMP_FB: C12.1, R13.1, R14.1, U3.2 (-)
- new net AMP_INP: C11.1, R12.2, U3.3 (+)
- new net AMP_OUT: C12.2, R13.2, R15.1, U3.1
- new net CP_RST: R42.2, U6.9 (~{RST})
- new net CP_VBUS: R40.2, R41.1, U6.8 (VBUS)
- new net CP_VDD: C42.1, C43.1, R42.1, U6.6 (VDD)
- new net DAC_BCK: R34.2, U7.13 (BCK)
- new net DAC_CAPM: C55.2, U7.4 (CAPM)
- new net DAC_CAPP: C55.1, U7.2 (CAPP)
- new net DAC_DIN: R36.2, U7.14 (DIN)
- new net DAC_LDOO: C57.1, U7.18 (LDOO)
- new net DAC_LRCK: R35.2, U7.15 (LRCK)
- new net DAC_OUTL: R51.1, U7.6 (OUTL)
- new net DAC_OUTR: R52.1, U7.7 (OUTR)
- new net DAC_VNEG: C56.1, U7.5 (VNEG)
- new net DAC_XSMT: R50.2, U7.17 (XSMT)
- new net GAIN_LEG: C13.1, R14.2
- new net GNDA: C11.2, C13.2, C15.2, C16.2, C17.2, C18.2, C5.2, C6.2, D2.1 (A), J2.S, NT1.2, R10.2, R19.2, U3.11 (V-)
- new net IN_AC: C10.1, R11.1, R12.1
- new net IN_TIP: C10.2, J2.T, R10.1
- new net LED_PWR: D1.2 (A), R3.2
- new net LED_STAT: D3.2 (A), R24.2
- new net LINE_L: C58.1, J3.T, R51.2
- new net LINE_R: C59.1, J3.R, R52.2
- new net OPB_OUT: U3.6 (-), U3.7
- new net OPD_OUT: U3.13 (-), U3.14
- new net Q1_B: Q1.1 (B), R32.2
- new net Q2_B: Q2.1 (B), R33.2
- new net SK_INP: C15.1, R16.2, U3.10 (+)
- new net SK_MID: C14.1, R15.2, R16.1
- new net UART_DTR: Q2.2 (E), R32.1, U6.28 (~{DTR})
- new net UART_RTS: Q1.2 (E), R33.1, U6.24 (~{RTS})
- new net USB_CC1: J1.A5 (CC1), R1.1
- new net USB_CC2: J1.B5 (CC2), R2.1
- new net USB_DN: J1.A7 (D-), J1.B7 (D-), U4.3 (I/O2), U4.4 (I/O2), U6.5 (D-)
- new net USB_DP: J1.A6 (D+), J1.B6 (D+), U4.1 (I/O1), U4.6 (I/O1), U6.4 (D+)
- new net VBIAS: C17.1, R11.2, R18.2, R19.1, U3.12 (+), U3.5 (+)
- new net VBUS: F1.1, J1.A4 (VBUS), J1.A9 (VBUS), J1.B4 (VBUS), J1.B9 (VBUS), R40.1, U4.5 (VBUS)
- no-connect marks 0 -> 64
Other:
- note added: "(Butterworth) for the 48 kHz ADC. D2 clamps PA0 to 0..3.3 V."
- note added: "(GPIO43/44). Arduino: set 'USB CDC On Boot: Disabled' so"
- note added: "(half of VDDA) so the output centres on ADC mid-scale."
- note added: "1. Single 5 V supply from USB-C (laptop). CC1/CC2 5.1k pull-"
- note added: "2. USB data goes to the CP2102N only -> ESP32 UART0"
- note added: "3. STM32 is flashed over SWD (J4) with an external ST-Link. J4"
- note added: "4. Preamp runs single-supply 0-5 V (+5VA). VBIAS = 1.65 V"
- note added: "5. Stage A gain = 1 + 3k/220R = 14.6 (LTspice"
- note added: "6. Stage C = unity-gain Sallen-Key low-pass, fc ~ 15.8 kHz"
- note added: "6.35 mm input, TL974 single-supply preamp (1.65 V bias), anti-alias filter, ADC protection"
- note added: "7. GNDA (preamp) joins GND at NT1 only. Place NT1 near the"
- note added: "8. STM32 UFQFPN-32 exposed pad and ESP32 EPAD: connect to GND"
- note added: "ADC capture (PA0) + SAI1 I2S master to ESP32, SWD programming header"
- note added: "ANALOGUE FRONT END"
- note added: "CP2102N USB-UART BRIDGE"
- note added: "DESIGN NOTES"
- note added: "ESP32-S3-WROOM-1-N8"
- note added: "GuitarLineInV2Alt). Input clips above ~110 mV peak; raise R14"
- note added: "I2S (FMT=0), internal PLL (SCK=GND), RC output filter, 6.35 mm line out"
- note added: "I2S RX from STM32, I2S TX to DAC, UART0 to CP2102N, auto-reset / boot"
- note added: "PCM5102A DAC"
- note added: "POWER INPUT"
- note added: "STM32 VSSA/VSS pins in layout."
- note added: "STM32L432KCU6"
- note added: "Serial = UART0."
- note added: "USB-C 5 V (laptop), ESD, polyfuse, 3.3 V LDO, filtered preamp rail"
- note added: "bus powered, ESP32 UART0 + DTR/RTS auto-reset"
- note added: "downs = UFP sink, 500 mA default budget."
- note added: "for hotter sources."
- note added: "in the footprint."
- note added: "pin order: 1 VDD, 2 SWCLK, 3 GND, 4 SWDIO, 5 NRST, 6 SWO."
- company: (none) -> Sonido
- title: (none) -> Stanza Board - Guitar In / STM32 / ESP32-S3 / PCM5102A
- moved on the sheet: U1A, U2
